File: EAGLE/mainboard.brd (EAGLE design)
At the start: 62.2 x 63.2 mm, 16 parts, among them IC1 7805TV

Commit message: * Moved all EAGLE files into the project * Removed old copy-pasted boards * Updated .gitignore
Parts:
- removed ANALOG, DIGITAL: (no value), pinhead:1X15
- added ARDUINO_NANO1: (no value), ArduinoNanoV30:ARDUINO_NANO
- moved FRONT_PANEL_DATA 15.2 mm to (31.8, 53.3), turned to 0 degrees
- moved FRONT_PANEL_PWR 12.7 mm to (17.8, 53.3), turned to 0 degrees
- moved RXTX 1.27 mm to (52.1, 53.3)
Connections:
- removed net REB_A: DIGITAL.14, FRONT_PANEL_DATA.3
- removed net REB_B: DIGITAL.5, FRONT_PANEL_DATA.5
- removed net REB_SWITCH: DIGITAL.6, FRONT_PANEL_DATA.4
- removed net RXD: DIGITAL.2, RXTX.1
- removed net SCL: ANALOG.9, FRONT_PANEL_DATA.2
- removed net SDA: ANALOG.8, FRONT_PANEL_DATA.1
- removed net TXD: DIGITAL.1, RXTX.2
- new net A4/SDA: ARDUINO_NANO1.8, FRONT_PANEL_DATA.2
- new net A5/SCL: ARDUINO_NANO1.9, FRONT_PANEL_DATA.1
- new net D0/RX: ARDUINO_NANO1.17, RXTX.2
- new net D1/TX: ARDUINO_NANO1.16, RXTX.1
- new net D11/REB_A: ARDUINO_NANO1.29, FRONT_PANEL_DATA.3
- new net D2/REB_B: ARDUINO_NANO1.20, FRONT_PANEL_DATA.5
- new net D3/REB_SWITCH: ARDUINO_NANO1.21, FRONT_PANEL_DATA.4
- new net VIN: ARDUINO_NANO1.15
- net +5V: now also ARDUINO_NANO1.12; no longer ANALOG.12
- net A6: now also ARDUINO_NANO1.10; no longer ANALOG.10
- net A7: now also ARDUINO_NANO1.11; no longer ANALOG.11
- net D10: now also ARDUINO_NANO1.28; no longer DIGITAL.13
- net D4: now also ARDUINO_NANO1.22; no longer DIGITAL.7
- net D5: now also ARDUINO_NANO1.23; no longer DIGITAL.8
- net D6: now also ARDUINO_NANO1.24; no longer DIGITAL.9
- net D7: now also ARDUINO_NANO1.25; no longer DIGITAL.10
- net D8: now also ARDUINO_NANO1.26; no longer DIGITAL.11
- net D9: now also ARDUINO_NANO1.27; no longer DIGITAL.12
- net GND: now also ARDUINO_NANO1.14, ARDUINO_NANO1.19; no longer ANALOG.14, DIGITAL.4
Routing:
- net REB_A: track 61.8 -> 0.00 mm
- net REB_B: track 47.2 -> 0.00 mm
- net D11/REB_A: track 0.00 -> 46.0 mm
- net REB_SWITCH: track 45.2 -> 0.00 mm
- net SDA: track 34.5 -> 0.00 mm
- net SCL: track 33.3 -> 0.00 mm
- net A4/SDA: track 0.00 -> 27.5 mm
- net A5/SCL: track 0.00 -> 25.0 mm
- net D3/REB_SWITCH: track 0.00 -> 23.9 mm
- net TXD: track 20.0 -> 0.00 mm
- net D2/REB_B: track 0.00 -> 19.6 mm
- net D0/RX: track 0.00 -> 17.7 mm
- net RXD: track 16.1 -> 0.00 mm
- net D1/TX: track 0.00 -> 13.3 mm
- net +5V: track 68.8 -> 66.1 mm
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Other:
- board text added: "ANALOG_A"
- board text added: "ANALOG_B"
- board text added: "ARDUINO_NANO1"
- board text added: "C3"
- board text added: "C4"
- board text added: "DIGITAL_A"
- board text added: "DIGITAL_B"
- board text added: "DIGITAL_C"
- board text added: "FRONT_PANEL_DATA"
- board text added: "FRONT_PANEL_PWR"
- board text added: "IC1"
- board text added: "MOTOR_A"
- board text added: "MOTOR_B"
- board text added: "PWR"
- board text added: "RXTX"
